File: smoothie_sw_encoder/smoothie_sw_encoder.kicad_pcb (KiCad board)
At the start: 2 copper layers, 5 parts, among them P1 CONN_5, P2 CONN_2, SW1 SW_PUSH

Commit message: knob
Routing:
- net N-000007: track 59.5 -> 65.5 mm
Changed lines of the file:
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@@
   (general
     (links 11)
-    (no_connects 3)
+    (no_connects 2)
     (area 94.18873 85.949999 118.050001 126.050001)
     (thickness 1.6)
     (drawings 4)
-    (tracks 33)
+    (tracks 35)
     (zones 0)
     (modules 5)
@@
   (segment (start 104.19 88.46) (end 99.27 88.46) (width 1) (layer Dessous.Cu) (net 6))
   (segment (start 99.27 88.46) (end 98 89.73) (width 1) (layer Dessous.Cu) (net 6))
+  (segment (start 110.5 107) (end 116.5 107) (width 1) (layer Dessous.Cu) (net 7) (status 400000))
   (segment (start 102.92 101) (end 103 101) (width 1) (layer Dessous.Cu) (net 7))
   (segment (start 108 123) (end 108 121.5) (width 1) (layer Dessous.Cu) (net 7))
@@
   (segment (start 112 124) (end 109 124) (width 1) (layer Dessous.Cu) (net 7))
   (segment (start 116.5 119.5) (end 112 124) (width 1) (layer Dessous.Cu) (net 7))
-  (segment (start 116.5 100) (end 116.5 119.5) (width 1) (layer Dessous.Cu) (net 7))
+  (segment (start 116.5 100) (end 116.5 107) (width 1) (layer Dessous.Cu) (net 7))
+  (segment (start 116.5 107) (end 116.5 119.5) (width 1) (layer Dessous.Cu) (net 7))
   (segment (start 114 97.5) (end 116.5 100) (width 1) (layer Dessous.Cu) (net 7))
   (segment (start 106.5 97.5) (end 114 97.5) (width 1) (layer Dessous.Cu) (net 7))
